File: PCB/wiznet.kicad_sch (KiCad schematic)
At the start: 41 parts, among them IC3 W5100S-L, J3 2250056-1, Y2 25M

Commit message: change leds to mouser
Parts:
- D1, D2, D3, D4, D5: LCSC C118334 -> (none); mouser (none) -> https://eu.mouser.com/ProductDetail/LITEON/LTST-C194KGKT?qs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
Changed lines of the file:
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@@
 			)
 		)
-		(property "Datasheet" "~"
+		(property "Datasheet" "https://eu.mouser.com/datasheet/3/281/1/LTST_C194KGKT.PDF"
 			(at 43.18 50.8 0)
 			(effects
@@
 			)
 		)
-		(property "LCSC" "C118334"
+		(property "LCSC" ""
 			(at 43.18 50.8 90)
 			(effects
@@
 		(property "Sim.Pins" "1=K 2=A"
 			(at 43.18 50.8 0)
+			(effects
+				(font
+					(size 1.27 1.27)
+				)
+				(hide yes)
+			)
+		)
+		(property "mouser" "https://eu.mouser.com/ProductDetail/LITEON/LTST-C194KGKT?qs=xIkB7y1OToqWwFdcevEBdQ%3D%3D"
+			(at 43.18 50.8 90)
 			(effects
 				(font
@@
 			)
 		)
-		(property "Datasheet" "~"
+		(property "Datasheet" "https://eu.mouser.com/datasheet/3/281/1/LTST_C194KGKT.PDF"
 			(at 90.17 50.8 0)
 			(effects
@@
 			)
 		)
-		(property "LCSC" "C118334"
+		(property "LCSC" ""
 			(at 90.17 50.8 90)
 			(effects
@@
 		(property "Sim.Pins" "1=K 2=A"
 			(at 90.17 50.8 0)
+			(effects
+				(font
+					(size 1.27 1.27)
+				)
+				(hide yes)
+			)
+		)
+		(property "mouser" "https://eu.mouser.com/ProductDetail/LITEON/LTST-C194KGKT?qs=xIkB7y1OToqWwFdcevEBdQ%3D%3D"
+			(at 90.17 50.8 90)
 			(effects
 				(font
@@
 			)
 		)
-		(property "Datasheet" "~"
+		(property "Datasheet" "https://eu.mouser.com/datasheet/3/281/1/LTST_C194KGKT.PDF"
 			(at 124.46 50.8 0)
 			(effects
@@
 			)
 		)
-		(property "LCSC" "C118334"
+		(property "LCSC" ""
 			(at 124.46 50.8 90)
 			(effects
@@
 		(property "Sim.Pins" "1=K 2=A"
 			(at 124.46 50.8 0)
+			(effects
+				(font
+					(size 1.27 1.27)
+				)
+				(hide yes)
+			)
+		)
+		(property "mouser" "https://eu.mouser.com/ProductDetail/LITEON/LTST-C194KGKT?qs=xIkB7y1OToqWwFdcevEBdQ%3D%3D"
+			(at 124.46 50.8 90)
 			(effects
 				(font
@@
 			)
 		)
-		(property "Datasheet" "~"
+		(property "Datasheet" "https://eu.mouser.com/datasheet/3/281/1/LTST_C194KGKT.PDF"
 			(at 60.96 50.8 0)
 			(effects
@@
 			)
 		)
-		(property "LCSC" "C118334"
+		(property "LCSC" ""
 			(at 60.96 50.8 90)
 			(effects
@@
 		(property "Sim.Pins" "1=K 2=A"
 			(at 60.96 50.8 0)
+			(effects
+				(font
+					(size 1.27 1.27)
+				)
+				(hide yes)
+			)
+		)
+		(property "mouser" "https://eu.mouser.com/ProductDetail/LITEON/LTST-C194KGKT?qs=xIkB7y1OToqWwFdcevEBdQ%3D%3D"
+			(at 60.96 50.8 90)
 			(effects
 				(font
@@
 			)
 		)
-		(property "Datasheet" "~"
+		(property "Datasheet" "https://eu.mouser.com/datasheet/3/281/1/LTST_C194KGKT.PDF"
 			(at 26.67 50.8 0)
 			(effects
@@
 			)
 		)
-		(property "LCSC" "C118334"
+		(property "LCSC" ""
 			(at 26.67 50.8 90)
 			(effects
@@
 			(effects
 				(font
+					(size 1.27 1.27)
+				)
+				(hide yes)
+			)
+		)
+		(property "mouser" "https://eu.mouser.com/ProductDetail/LITEON/LTST-C194KGKT?qs=xIkB7y1OToqWwFdcevEBdQ%3D%3D"
+			(at 26.67 50.8 90)
+			(effects
+				(font
