File: PCB/design.kicad_pcb (KiCad board)
At the start: 4 copper layers, 78.8 x 38.5 mm, 66 parts, among them IC3 W5100S-L, J1 BNC, J2 BNC, J3 2250056-1, U1 MCP6002-xMC, U2 MCP6002-xMC, U3 NUCLEO-L432KC, Y2 25M

Commit message: add channel silkscreen labels
Other:
- board text added: "CH0"
- board text added: "CH1"
Changed lines of the file:
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@@
+		)
+	)
+	(gr_text "CH0"
+		(at 101.752 65.488 90)
+		(layer "F.SilkS" knockout)
+		(effects
+			(font
+				(size 2 2)
+				(thickness 0.375)
+				(bold yes)
+			)
+			(justify right top)
+		)
+	)
+	(gr_text "CH1"
+		(at 114.686 65.48 90)
+		(layer "F.SilkS" knockout)
+		(effects
+			(font
+				(size 2 2)
+				(thickness 0.375)
+				(bold yes)
+			)
+			(justify right bottom)
 		)
 	)
